Commit message: add meshes

File: src/base_movement/urdf/base/abluo_body.urdf.xacro (robot description, xacro)
@@ -22,5 +22,5 @@
         <origin xyz="0 0 0.02" rpy="0 0 0" />
         <geometry>
-          <mesh filename="package://abluo_base_description/meshes/base_link.STL" />
+          <mesh filename="package://base_movement/meshes/base_link.STL" />
         </geometry>
         <material name="custom">
@@ -31,5 +31,5 @@
         <origin xyz="0 0 0.02" rpy="0 0 0" />
         <geometry>
-          <mesh filename="package://abluo_base_description/meshes/base_link.STL" />
+          <mesh filename="package://base_movement/meshes/base_link.STL" />
         </geometry>
       </collision>

File: src/base_movement/urdf/sensors/rplidar.gazebo.xacro (robot description, xacro)
@@ -11,5 +11,5 @@
                 <origin xyz="0 0 0" rpy="0 0 0" />
                 <geometry>
-                    <mesh filename="package://abluo_base_description/meshes/lidar.STL" />
+                    <mesh filename="package://base_movement/meshes/lidar.STL" />
                 </geometry>
                 <material name="">
@@ -20,5 +20,5 @@
                 <origin xyz="0 0 0" rpy="0 0 0" />
                 <geometry>
-                    <mesh filename="package://abluo_base_description/meshes/lidar.STL" />
+                    <mesh filename="package://base_movement/meshes/lidar.STL" />
                 </geometry>
             </collision>
@@ -72,5 +72,5 @@
                 <origin xyz="0 0 0" rpy="0 0 0" />
                 <geometry>
-                    <mesh filename="package://abluo_base_description/meshes/camera.STL" />
+                    <mesh filename="package://base_movement/meshes/camera.STL" />
                 </geometry>
                 <material name="">
@@ -81,5 +81,5 @@
                 <origin xyz="0 0 0" rpy="0 0 0" />
                 <geometry>
-                    <mesh filename="package://abluo_base_description/meshes/camera.STL" />
+                    <mesh filename="package://base_movement/meshes/camera.STL" />
                 </geometry>
             </collision>

File: src/base_movement/urdf/wheels/omni_wheel.urdf.xacro (robot description, xacro)
@@ -25,10 +25,10 @@
         <xacro:if value="${reflect}">
           <geometry>
-            <mesh filename="package://abluo_base_description/meshes/front_left_w.STL" />
+            <mesh filename="package://base_movement/meshes/front_left_w.STL" />
           </geometry>
           </xacro:if>
           <xacro:unless value="${reflect}">
             <geometry>
-              <mesh filename="package://abluo_base_description/meshes/front_right_w.STL" />
+              <mesh filename="package://base_movement/meshes/front_right_w.STL" />
             </geometry>
 		    </xacro:unless>
